Commit message: Added frames in the package 'h1_description'

File: h1_description/urdf/h1_with_hand.urdf (robot description, URDF)
Before this commit: robot h1, 52 links, 51 joints
Links:
- added link imu_link
Joints:
- added joint imu_joint: type fixed, parent torso_link, child imu_link, origin xyz=-0.04452 -0.01891 0.27756 rpy=0 0 0
